File: IonSensorRevC - JST.sch (EAGLE design)
At the start: 19 parts, among them U1 REF2033AIDDCT, U2 INA826AIDR, U3 INA826AIDR, U4 INA826AIDR, X1 B4B-PH-K-S

Commit message: Update traces
Updated traces to minimize noise
Parts:
- X1: value B4B-PH-K-S -> B5B-XH-2; device con-JST PH:B4B-PH-K-S -> con-JST XH:B5B-XH-2
Connections:
- removed net A1: MS1.GPIOA1
- removed net A3: MS1.GPIOA3
- removed net A5: MS1.GPIOA5
- removed net CH1: U3.+IN, X1.2
- new net CH4: U4.+IN, X1.2
- net CH0: now also X1.4; no longer X1.3
- net CH2: now also U3.+IN, X1.3; no longer U4.+IN, X1.1
- net GND: now also MS1.GPIOA1, MS1.GPIOA3, MS1.GPIOA5
- net REF: now also X1.5; no longer X1.4
- net VCC/2: now also X1.1
Other:
- note added: "C"
Changed lines of the file:
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@@
 <part name="R4" library="adafruit" library_urn="urn:adsk.eagle:library:420" deviceset="R-US_" device="R0402" package3d_urn="urn:adsk.eagle:package:6240564/1" value="10k"/>
 <part name="P+7" library="supply1" library_urn="urn:adsk.eagle:library:371" deviceset="VCC/2" device=""/>
-<part name="X1" library="con-JST PH" deviceset="B4B-PH" device="-K-S"/>
+<part name="X1" library="con-JST XH" deviceset="B5B-XH" device="-2"/>
+<part name="P+8" library="supply1" library_urn="urn:adsk.eagle:library:371" deviceset="VCC/2" device=""/>
 </parts>
 <sheets>
 <sheet>
 <plain>
+<text x="238.76" y="7.62" size="2.54" layer="94">C</text>
 </plain>
 <instances>
@@
 <attribute name="VALUE" x="124.46" y="27.94" size="1.778" layer="96" rot="R90"/>
 </instance>
-<instance part="X1" gate="G$1" x="81.28" y="25.4" smashed="yes" rot="MR180">
-<attribute name="VALUE" x="80.01" y="35.56" size="1.778" layer="96" rot="MR180"/>
-<attribute name="NAME" x="80.01" y="19.558" size="1.778" layer="95" rot="MR180"/>
+<instance part="X1" gate="G$1" x="66.04" y="33.02" smashed="yes">
+<attribute name="VALUE" x="64.77" y="22.86" size="1.778" layer="96"/>
+<attribute name="NAME" x="64.77" y="41.402" size="1.778" layer="95"/>
+</instance>
+<instance part="P+8" gate="G$1" x="86.36" y="40.64" smashed="yes">
+<attribute name="VALUE" x="83.82" y="38.1" size="1.778" layer="96" rot="R90"/>
 </instance>
 </instances>
@@
 <wire x1="58.42" y1="144.78" x2="55.88" y2="144.78" width="0.1524" layer="91"/>
 <pinref part="GND1" gate="1" pin="GND"/>
-<wire x1="55.88" y1="144.78" x2="55.88" y2="109.22" width="0.1524" layer="91"/>
+<wire x1="55.88" y1="144.78" x2="55.88" y2="139.7" width="0.1524" layer="91"/>
+<pinref part="MS1" gate="G$1" pin="GPIOA1"/>
+<wire x1="55.88" y1="139.7" x2="55.88" y2="134.62" width="0.1524" layer="91"/>
+<wire x1="55.88" y1="134.62" x2="55.88" y2="129.54" width="0.1524" layer="91"/>
+<wire x1="55.88" y1="129.54" x2="55.88" y2="109.22" width="0.1524" layer="91"/>
+<wire x1="58.42" y1="139.7" x2="55.88" y2="139.7" width="0.1524" layer="91"/>
+<junction x="55.88" y="139.7"/>
+<pinref part="MS1" gate="G$1" pin="GPIOA3"/>
+<wire x1="58.42" y1="134.62" x2="55.88" y2="134.62" width="0.1524" layer="91"/>
+<junction x="55.88" y="134.62"/>
+<pinref part="MS1" gate="G$1" pin="GPIOA5"/>
+<wire x1="58.42" y1="129.54" x2="55.88" y2="129.54" width="0.1524" layer="91"/>
+<junction x="55.88" y="129.54"/>
 </segment>
 <segment>
@@
 </segment>
 </net>
-<net name="A1" class="0">
-<segment>
-<pinref part="MS1" gate="G$1" pin="GPIOA1"/>
-<wire x1="53.34" y1="139.7" x2="58.42" y2="139.7" width="0.1524" layer="91"/>
-<label x="53.34" y="139.7" size="1.27" layer="95" rot="R180" xref="yes"/>
-</segment>
-</net>
 <net name="A2" class="0">
 <segment>
@@
 </segment>
 </net>
-<net name="A3" class="0">
-<segment>
-<pinref part="MS1" gate="G$1" pin="GPIOA3"/>
-<wire x1="53.34" y1="134.62" x2="58.42" y2="134.62" width="0.1524" layer="91"/>
-<label x="53.34" y="134.62" size="1.27" layer="95" rot="R180" xref="yes"/>
-</segment>
-</net>
 <net name="A4" class="0">
 <segment>
@@
 <wire x1="175.26" y1="73.66" x2="172.72" y2="73.66" width="0.1524" layer="91"/>
 <label x="175.26" y="73.66" size="1.016" layer="95" xref="yes"/>
-</segment>
-</net>
-<net name="A5" class="0">
-<segment>
-<pinref part="MS1" gate="G$1" pin="GPIOA5"/>
-<wire x1="53.34" y1="129.54" x2="58.42" y2="129.54" width="0.1524" layer="91"/>
-<label x="53.34" y="129.54" size="1.27" layer="95" rot="R180" xref="yes"/>
 </segment>
 </net>
@@
 <wire x1="127" y1="25.4" x2="127" y2="27.94" width="0.1524" layer="91"/>
 </segment>
+<segment>
+<pinref part="P+8" gate="G$1" pin="VCC/2"/>
+<pinref part="X1" gate="G$1" pin="1"/>
+<wire x1="86.36" y1="38.1" x2="86.36" y2="27.94" width="0.1524" layer="91"/>
+<wire x1="86.36" y1="27.94" x2="73.66" y2="27.94" width="0.1524" layer="91"/>
+</segment>
 </net>
 <net name="N$1" class="0">
@@
 </segment>
 <segment>
-<pinref part="X1" gate="G$1" pin="4"/>
-<wire x1="91.44" y1="22.86" x2="88.9" y2="22.86" width="0.1524" layer="91"/>
-<label x="91.44" y="22.86" size="1.016" layer="95" xref="yes"/>
+<pinref part="X1" gate="G$1" pin="5"/>
+<wire x1="76.2" y1="38.1" x2="73.66" y2="38.1" width="0.1524" layer="91"/>
+<label x="76.2" y="38.1" size="1.27" layer="95" xref="yes"/>
 </segment>
 </net>
@@
 </segment>
 <segment>
-<pinref part="X1" gate="G$1" pin="3"/>
-<wire x1="91.44" y1="25.4" x2="88.9" y2="25.4" width="0.1524" layer="91"/>
-<label x="91.44" y="25.4" size="1.016" layer="95" xref="yes"/>
-</segment>
-</net>
-<net name="CH1" class="0">
+<pinref part="X1" gate="G$1" pin="4"/>
+<wire x1="76.2" y1="35.56" x2="73.66" y2="35.56" width="0.1524" layer="91"/>
+<label x="76.2" y="35.56" size="1.27" layer="95" xref="yes"/>
+</segment>
+</net>
+<net name="CH2" class="0">
 <segment>
 <pinref part="U3" gate="G$1" pin="+IN"/>
@@
 </segment>
 <segment>
-<pinref part="X1" gate="G$1" pin="2"/>
-<wire x1="91.44" y1="27.94" x2="88.9" y2="27.94" width="0.1524" layer="91"/>
-<label x="91.44" y="27.94" size="1.016" layer="95" xref="yes"/>
-</segment>
-</net>
-<net name="CH2" class="0">
+<pinref part="X1" gate="G$1" pin="3"/>
+<wire x1="76.2" y1="33.02" x2="73.66" y2="33.02" width="0.1524" layer="91"/>
+<label x="76.2" y="33.02" size="1.27" layer="95" xref="yes"/>
+</segment>
+</net>
+<net name="CH4" class="0">
 <segment>
 <pinref part="U4" gate="G$1" pin="+IN"/>
@@
 </segment>
 <segment>
-<pinref part="X1" gate="G$1" pin="1"/>
-<wire x1="91.44" y1="30.48" x2="88.9" y2="30.48" width="0.1524" layer="91"/>
-<label x="91.44" y="30.48" size="1.016" layer="95" xref="yes"/>
-</segment>
-</net>
+<pinref part="X1" gate="G$1" pin="2"/>
+<wire x1="76.2" y1="30.48" x2="73.66" y2="30.48" width="0.1524" layer="91"/>
+<label x="76.2" y="30.48" size="1.27" layer="95" xref="yes"/>
+</segment>
+</net>
