File: IonSensor.brd (EAGLE design)
At the start: 50.8 x 22.9 mm, 21 parts, among them IC1 QUAD_OPAMPD, IC2 QUAD_OPAMPD, IC3 QUAD_OPAMPD, X1 JST-XH-04-PIN-LONG-PAD

Commit message: Fixed wiring
Made sure it's a differential amplifier!
Removed R13.
Parts:
- removed R13: 10k, rcl:R0603
Connections:
- net CH0: no longer R1.1
- net CH1: no longer R5.1
- net CH2: no longer R9.1
- net GND: now also R1.1, R5.1, R9.1; no longer R13.2
- net REF: no longer R13.1
Routing:
- net REF: track 59.2 -> 48.2 mm, vias 4 -> 3
- net CH2: track 12.5 -> 9.42 mm
- net CH1: track 26.2 -> 23.2 mm
- net CH0: track 40.0 -> 36.9 mm
Changed lines of the file:
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@@
 </element>
 <element name="X1" library="Rembrandt Electronics - JST XH Connectors v1-0" package="JST-XH-04-PACKAGE-LONG-PAD" value="JST-XH-04-PIN-LONG-PAD" x="46.99" y="11.43" smashed="yes" rot="R270"/>
-<element name="R13" library="rcl" library_urn="urn:adsk.eagle:library:334" package="R0603" package3d_urn="urn:adsk.eagle:package:23555/3" value="10k" x="3.81" y="11.43" smashed="yes" rot="R270">
-<attribute name="NAME" x="4.826" y="9.906" size="0.6096" layer="25" rot="R180"/>
-<attribute name="POPULARITY" value="77" x="3.81" y="11.43" size="1.778" layer="27" ratio="15" rot="R270" display="off"/>
-<attribute name="SPICEPREFIX" value="R" x="3.81" y="11.43" size="1.778" layer="27" ratio="15" rot="R270" display="off"/>
-<attribute name="VALUE" x="2.794" y="12.954" size="0.6096" layer="27"/>
-</element>
 </elements>
 <signals>
@@
 <contactref element="C2" pad="2"/>
 <contactref element="C1" pad="2"/>
-<contactref element="R13" pad="2"/>
+<contactref element="R1" pad="1"/>
+<contactref element="R5" pad="1"/>
+<contactref element="R9" pad="1"/>
 </signal>
 <signal name="+3V3">
@@
 <signal name="CH0">
 <contactref element="IC1" pad="3"/>
-<contactref element="R1" pad="1"/>
-<wire x1="13.97" y1="14.5034" x2="13.97" y2="17.565" width="0.381" layer="1"/>
 <wire x1="13.97" y1="14.5034" x2="13.97" y2="12.7" width="0.381" layer="1"/>
 <via x="13.97" y="12.7" extent="1-16" drill="0.381"/>
@@
 <signal name="CH1">
 <contactref element="IC2" pad="3"/>
-<contactref element="R5" pad="1"/>
-<wire x1="26.67" y1="17.565" x2="26.67" y2="14.5034" width="0.381" layer="1"/>
 <wire x1="26.67" y1="14.5034" x2="26.67" y2="12.7" width="0.381" layer="1"/>
 <via x="26.67" y="12.7" extent="1-16" drill="0.381"/>
@@
 <signal name="CH2">
 <contactref element="IC3" pad="3"/>
-<contactref element="R9" pad="1"/>
-<wire x1="39.37" y1="14.5034" x2="39.37" y2="17.565" width="0.381" layer="1"/>
 <wire x1="39.37" y1="14.5034" x2="39.37" y2="12.7" width="0.381" layer="1"/>
 <via x="39.37" y="12.7" extent="1-16" drill="0.381"/>
@@
 <contactref element="IC1" pad="5"/>
 <contactref element="IC2" pad="5"/>
-<contactref element="R13" pad="1"/>
 <wire x1="11.43" y1="14.5034" x2="11.43" y2="12.7" width="0.381" layer="1"/>
 <via x="11.43" y="12.7" extent="1-16" drill="0.381"/>
@@
 <wire x1="36.83" y1="14.5034" x2="36.83" y2="12.7" width="0.381" layer="1"/>
 <via x="36.83" y="12.7" extent="1-16" drill="0.381"/>
-<wire x1="3.81" y1="12.28" x2="3.81" y2="15.24" width="0.381" layer="1"/>
-<via x="3.81" y="15.24" extent="1-16" drill="0.381"/>
-<wire x1="3.81" y1="15.24" x2="11.43" y2="15.24" width="0.381" layer="16"/>
-<wire x1="11.43" y1="15.24" x2="24.13" y2="15.24" width="0.381" layer="16"/>
+<wire x1="11.43" y1="12.7" x2="11.43" y2="14.605" width="0.381" layer="16"/>
+<wire x1="12.065" y1="15.24" x2="11.43" y2="14.605" width="0.381" layer="16"/>
+<wire x1="12.065" y1="15.24" x2="24.13" y2="15.24" width="0.381" layer="16"/>
 <wire x1="24.13" y1="15.24" x2="36.83" y2="15.24" width="0.381" layer="16"/>
-<wire x1="11.43" y1="12.7" x2="11.43" y2="15.24" width="0.381" layer="16"/>
 <wire x1="24.13" y1="12.7" x2="24.13" y2="15.24" width="0.381" layer="16"/>
 <wire x1="36.83" y1="12.7" x2="36.83" y2="15.24" width="0.381" layer="16"/>
