File: IonSensor.sch (EAGLE design)
At the start: 20 parts, among them IC1 QUAD_OPAMPD, IC2 QUAD_OPAMPD, IC3 QUAD_OPAMPD, X1 JST-XH-04-PIN-LONG-PAD

Commit message: Switch to 2 channel opamp
Switched to 2 channel opamp instead of quad opamp.
Parts:
- added C4, C5, C6, C7, C8, C9: 0.1uF, adafruit:C-USC0402
- added R13, R16: 1M, adafruit:R-US_R0402
- added R14, R17, R18: 10k, adafruit:R-US_R0402
- added R15: 20k, adafruit:R-US_R0402
- C1, C2, C3: device adafruit:C-USC0603 -> adafruit:C-USC0402
- IC1, IC2, IC3: value QUAD_OPAMPD -> LM358D; device adafruit:QUAD_OPAMPD -> linear:LM358D
- R1, R4: value 100k -> 1M; device adafruit:R-US_R0603 -> adafruit:R-US_R0402
- R10, R7: value 10k -> 1M; device adafruit:R-US_R0603 -> adafruit:R-US_R0402
- R11, R2, R6: device adafruit:R-US_R0603 -> adafruit:R-US_R0402
- R12, R5, R8: value 100k -> 10k; device adafruit:R-US_R0603 -> adafruit:R-US_R0402
- R3: value 10k -> 20k; device adafruit:R-US_R0603 -> adafruit:R-US_R0402
- R9: value 100k -> 20k; device adafruit:R-US_R0603 -> adafruit:R-US_R0402
- X1: value JST-XH-04-PIN-LONG-PAD -> B4B-XH-2; device Rembrandt Electronics - JST XH Connectors v1-0:JST-XH-04-PIN-LONG-PAD -> con-JST XH:B4B-XH-2
Connections:
- removed net N$13: IC3C.+IN, R10.2, R9.2
- removed net N$14: IC3C.-IN, R11.2, R12.1
- removed net REF: IC1B.+IN, IC2B.+IN, IC3B.+IN, X1-1.S
- new net A1: C2.1, MS1.GPIOA1, R4.2
- new net A3: C4.1, MS1.GPIOA3, R10.2
- new net A5: C6.1, MS1.GPIOA5, R16.2
- new net N$10: IC3A.OUT, R13.1, R15.2
- new net N$5: IC2A.-IN, R8.2, R9.1
- net +3V3: now also C7.1, C8.1, C9.1; no longer C1.1, C2.1, C3.1
- net A0: now also C1.1, R1.2; no longer IC1C.OUT, R4.2
- net A2: now also C3.1, R7.2; no longer IC2C.OUT, R8.2
- net A4: now also C5.1, R13.2; no longer IC3C.OUT, R12.2
- net CH0: now also IC1B.+IN, R2.1, X1.4; no longer IC1A.+IN, X1-4.S
- net CH1: now also IC2B.+IN, R8.1, X1.3; no longer IC2A.+IN, X1-3.S
- net CH2: now also IC3B.+IN, R14.1, X1.2; no longer IC3A.+IN, X1-2.S
- net GND: now also C4.2, C5.2, C6.2, C7.2, C8.2, C9.2, IC1A.+IN, IC2A.+IN, IC3A.+IN, R11.1, R17.1, X1.1; no longer R1.1, R9.1
- net N$1: now also R2.2, R3.1; no longer IC1A.OUT, R2.1
- net N$11: now also IC3B.-IN, R17.2, R18.1; no longer IC3A.-IN, IC3A.OUT, R10.1
- net N$12: now also R16.1, R18.2; no longer IC3B.-IN, R11.1
- net N$2: now also IC1B.-IN, R5.2, R6.1; no longer IC1C.+IN, R1.2, R2.2
- net N$3: now also IC1A.OUT, R1.1, R3.2; no longer IC1B.-IN, IC1B.OUT, R3.1
- net N$4: now also IC1B.OUT, R6.2; no longer IC1C.-IN, R3.2
- net N$6: now also R7.1, R9.2; no longer IC2A.-IN, R6.1
- net N$7: now also R11.2, R12.1; no longer IC2B.OUT, R7.1
- net N$8: now also IC2B.OUT, R10.1, R12.2; no longer IC2C.+IN, R5.2, R6.2
- net N$9: now also IC3A.-IN, R14.2, R15.1; no longer IC2C.-IN, R7.2, R8.1
Other:
- note added: "D"
- note removed: "A"
- moved on the sheet: C1, C2, C3, IC1A, IC1B, IC2A, IC2B, IC3A, IC3B, R1, R10, R11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

Commit message: Revert "Switch to 2 channel opamp"
This reverts commit d2c6276b5e9005aaa4bb267ec01d57cf95291150.
Parts:
- removed C4, C5, C6, C7, C8, C9: 0.1uF, adafruit:C-USC0402
- removed R13, R16: 1M, adafruit:R-US_R0402
- removed R14, R17, R18: 10k, adafruit:R-US_R0402
- removed R15: 20k, adafruit:R-US_R0402
- C1, C2, C3: device adafruit:C-USC0402 -> adafruit:C-USC0603
- IC1, IC2, IC3: value LM358D -> QUAD_OPAMPD; device linear:LM358D -> adafruit:QUAD_OPAMPD
- R1, R4: value 1M -> 100k; device adafruit:R-US_R0402 -> adafruit:R-US_R0603
- R10, R7: value 1M -> 10k; device adafruit:R-US_R0402 -> adafruit:R-US_R0603
- R11, R2, R6: device adafruit:R-US_R0402 -> adafruit:R-US_R0603
- R12, R5, R8: value 10k -> 100k; device adafruit:R-US_R0402 -> adafruit:R-US_R0603
- R3: value 20k -> 10k; device adafruit:R-US_R0402 -> adafruit:R-US_R0603
- R9: value 20k -> 100k; device adafruit:R-US_R0402 -> adafruit:R-US_R0603
- X1: value B4B-XH-2 -> JST-XH-04-PIN-LONG-PAD; device con-JST XH:B4B-XH-2 -> Rembrandt Electronics - JST XH Connectors v1-0:JST-XH-04-PIN-LONG-PAD
Connections:
- removed net A1: C2.1, MS1.GPIOA1, R4.2
- removed net A3: C4.1, MS1.GPIOA3, R10.2
- removed net A5: C6.1, MS1.GPIOA5, R16.2
- removed net N$10: IC3A.OUT, R13.1, R15.2
- removed net N$5: IC2A.-IN, R8.2, R9.1
- new net N$13: IC3C.+IN, R10.2, R9.2
- new net N$14: IC3C.-IN, R11.2, R12.1
- new net REF: IC1B.+IN, IC2B.+IN, IC3B.+IN, X1-1.S
- net +3V3: now also C1.1, C2.1, C3.1; no longer C7.1, C8.1, C9.1
- net A0: now also IC1C.OUT, R4.2; no longer C1.1, R1.2
- net A2: now also IC2C.OUT, R8.2; no longer C3.1, R7.2
- net A4: now also IC3C.OUT, R12.2; no longer C5.1, R13.2
- net CH0: now also IC1A.+IN, X1-4.S; no longer IC1B.+IN, R2.1, X1.4
- net CH1: now also IC2A.+IN, X1-3.S; no longer IC2B.+IN, R8.1, X1.3
- net CH2: now also IC3A.+IN, X1-2.S; no longer IC3B.+IN, R14.1, X1.2
- net GND: now also R1.1, R9.1; no longer C4.2, C5.2, C6.2, C7.2, C8.2, C9.2, IC1A.+IN, IC2A.+IN, IC3A.+IN, R11.1, R17.1, X1.1
- net N$1: now also IC1A.OUT, R2.1; no longer R2.2, R3.1
- net N$11: now also IC3A.-IN, IC3A.OUT, R10.1; no longer IC3B.-IN, R17.2, R18.1
- net N$12: now also IC3B.-IN, R11.1; no longer R16.1, R18.2
- net N$2: now also IC1C.+IN, R1.2, R2.2; no longer IC1B.-IN, R5.2, R6.1
- net N$3: now also IC1B.-IN, IC1B.OUT, R3.1; no longer IC1A.OUT, R1.1, R3.2
- net N$4: now also IC1C.-IN, R3.2; no longer IC1B.OUT, R6.2
- net N$6: now also IC2A.-IN, R6.1; no longer R7.1, R9.2
- net N$7: now also IC2B.OUT, R7.1; no longer R11.2, R12.1
- net N$8: now also IC2C.+IN, R5.2, R6.2; no longer IC2B.OUT, R10.1, R12.2
- net N$9: now also IC2C.-IN, R7.2, R8.1; no longer IC3A.-IN, R14.2, R15.1
Other:
- note added: "A"
- note removed: "D"
- moved on the sheet: C1, C2, C3, IC1A, IC1B, IC2A, IC2B, IC3A, IC3B, R1, R10, R11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

Commit message: Rev. D
Upgrade to Rev. D, no connector
Parts:
- removed X1: JST-XH-04-PIN-LONG-PAD, Rembrandt Electronics - JST XH Connectors v1-0:JST-XH-04-PIN-LONG-PAD
- added C4, C5, C6, C7, C8, C9: 0.1uF, adafruit:C-USC0402
- added R13, R17, R18, R22, R23, R27, R28: 10k, adafruit:R-US_R0402
- added R14, R16, R19, R21, R24, R26, R29: 100k, adafruit:R-US_R0402
- added R15, R20, R25, R30: 1M, adafruit:R-US_R0402
- C1, C2, C3: device adafruit:C-USC0603 -> adafruit:C-USC0402
- R1, R2, R3, R4, R7, R9: device adafruit:R-US_R0603 -> adafruit:R-US_R0402
- R10: value 10k -> 1M; device adafruit:R-US_R0603 -> adafruit:R-US_R0402
- R11, R6: value 10k -> 100k; device adafruit:R-US_R0603 -> adafruit:R-US_R0402
- R12, R8: value 100k -> 10k; device adafruit:R-US_R0603 -> adafruit:R-US_R0402
- R5: value 100k -> 1M; device adafruit:R-US_R0603 -> adafruit:R-US_R0402
Connections:
- removed net N$1 (its old number): IC1A.-IN, IC1A.OUT, R2.1
- new net A1: C2.1, MS1.GPIOA1, R10.2
- new net A3: C4.1, MS1.GPIOA3, R20.2
- new net A5: C6.1, MS1.GPIOA5, R30.2
- new net C1+: IC1A.-IN, IC1A.OUT, R2.1, R8.1
- new net C1-: IC1B.-IN, IC1B.OUT, R3.1, R7.1
- new net C2+: IC2A.-IN, IC2A.OUT, R12.1, R18.1
- new net C2-: IC2B.-IN, IC2B.OUT, R13.1, R17.1
- new net C3+: IC3A.-IN, IC3A.OUT, R22.1, R28.1
- new net C3-: IC3B.-IN, IC3B.OUT, R23.1, R27.1
- new net N$10: IC1D.OUT, R10.1, R9.2
- new net N$15: IC3D.-IN, R28.2, R29.1
- new net N$16: IC2D.OUT, R19.2, R20.1
- new net N$17: IC3C.OUT, R24.2, R25.1
- new net N$18: IC3D.OUT, R29.2, R30.1
- new net N$4: IC1D.+IN, R6.2, R7.2
- new net N$5: IC1C.OUT, R4.2, R5.1
- net +3V3: now also C7.1, C8.1, C9.1; no longer C1.1, C2.1, C3.1
- net A0: now also C1.1, R5.2; no longer IC1C.OUT, R4.2
- net A2: now also C3.1, R15.2; no longer IC2C.OUT, R8.2
- net A4: now also C5.1, R25.2; no longer IC3C.OUT, R12.2
- net CH0: no longer X1-4.S
- net CH1: no longer X1-3.S
- net CH2: no longer X1-2.S
- net GND: now also C4.2, C5.2, C6.2, C7.2, C8.2, C9.2, R11.1, R16.1, R21.1, R26.1, R6.1; no longer R5.1, R9.1
- net N$11: now also IC2D.+IN, R16.2, R17.2; no longer IC3A.-IN, IC3A.OUT, R10.1
- net N$12: now also IC3D.+IN, R26.2, R27.2; no longer IC3B.-IN, IC3B.OUT, R11.1
- net N$13: now also IC2D.-IN, R18.2, R19.1; no longer IC3C.+IN, R10.2, R9.2
- net N$14: now also IC2C.OUT, R14.2, R15.1; no longer IC3C.-IN, R11.2, R12.1
- net N$3: now also IC3C.+IN, R21.2, R22.2; no longer IC1B.-IN, IC1B.OUT, R3.1
- net N$6: now also IC1D.-IN, R8.2, R9.1; no longer IC2A.-IN, IC2A.OUT, R6.1
- net N$7: now also IC3C.-IN, R23.2, R24.1; no longer IC2B.-IN, IC2B.OUT, R7.1
- net N$8: now also R11.2, R12.2; no longer R5.2, R6.2
- net N$9: now also R13.2, R14.1; no longer R7.2, R8.1
- net REF: no longer X1-1.S
Other:
- note added: "D"
- note removed: "A"
- moved on the sheet: C1, C2, C3, IC1A, IC1B, IC1C, IC2A, IC2B, IC2C, IC3A, IC3B, IC3C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

Commit message: Revert "Rev. D"
This reverts commit b0cd00c38bcd6b0f7db002c888a5e278bdb202ce.
Parts:
- removed C4, C5, C6, C7, C8, C9: 0.1uF, adafruit:C-USC0402
- removed R13, R17, R18, R22, R23, R27, R28: 10k, adafruit:R-US_R0402
- removed R14, R16, R19, R21, R24, R26, R29: 100k, adafruit:R-US_R0402
- removed R15, R20, R25, R30: 1M, adafruit:R-US_R0402
- added X1: JST-XH-04-PIN-LONG-PAD, Rembrandt Electronics - JST XH Connectors v1-0:JST-XH-04-PIN-LONG-PAD
- C1, C2, C3: device adafruit:C-USC0402 -> adafruit:C-USC0603
- R1, R2, R3, R4, R7, R9: device adafruit:R-US_R0402 -> adafruit:R-US_R0603
- R10: value 1M -> 10k; device adafruit:R-US_R0402 -> adafruit:R-US_R0603
- R11, R6: value 100k -> 10k; device adafruit:R-US_R0402 -> adafruit:R-US_R0603
- R12, R8: value 10k -> 100k; device adafruit:R-US_R0402 -> adafruit:R-US_R0603
- R5: value 1M -> 100k; device adafruit:R-US_R0402 -> adafruit:R-US_R0603
Connections:
- removed net A1: C2.1, MS1.GPIOA1, R10.2
- removed net A3: C4.1, MS1.GPIOA3, R20.2
- removed net A5: C6.1, MS1.GPIOA5, R30.2
- removed net C1+: IC1A.-IN, IC1A.OUT, R2.1, R8.1
- removed net C1-: IC1B.-IN, IC1B.OUT, R3.1, R7.1
- removed net C2+: IC2A.-IN, IC2A.OUT, R12.1, R18.1
- removed net C2-: IC2B.-IN, IC2B.OUT, R13.1, R17.1
- removed net C3+: IC3A.-IN, IC3A.OUT, R22.1, R28.1
- removed net C3-: IC3B.-IN, IC3B.OUT, R23.1, R27.1
- removed net N$10: IC1D.OUT, R10.1, R9.2
- removed net N$15: IC3D.-IN, R28.2, R29.1
- removed net N$16: IC2D.OUT, R19.2, R20.1
- removed net N$17: IC3C.OUT, R24.2, R25.1
- removed net N$18: IC3D.OUT, R29.2, R30.1
- removed net N$4 (its old number): IC1D.+IN, R6.2, R7.2
- removed net N$5: IC1C.OUT, R4.2, R5.1
- new net N$1: IC1A.-IN, IC1A.OUT, R2.1
- net +3V3: now also C1.1, C2.1, C3.1; no longer C7.1, C8.1, C9.1
- net A0: now also IC1C.OUT, R4.2; no longer C1.1, R5.2
- net A2: now also IC2C.OUT, R8.2; no longer C3.1, R15.2
- net A4: now also IC3C.OUT, R12.2; no longer C5.1, R25.2
- net CH0: now also X1-4.S
- net CH1: now also X1-3.S
- net CH2: now also X1-2.S
- net GND: now also R5.1, R9.1; no longer C4.2, C5.2, C6.2, C7.2, C8.2, C9.2, R11.1, R16.1, R21.1, R26.1, R6.1
- net N$11: now also IC3A.-IN, IC3A.OUT, R10.1; no longer IC2D.+IN, R16.2, R17.2
- net N$12: now also IC3B.-IN, IC3B.OUT, R11.1; no longer IC3D.+IN, R26.2, R27.2
- net N$13: now also IC3C.+IN, R10.2, R9.2; no longer IC2D.-IN, R18.2, R19.1
- net N$14: now also IC3C.-IN, R11.2, R12.1; no longer IC2C.OUT, R14.2, R15.1
- net N$3: now also IC1B.-IN, IC1B.OUT, R3.1; no longer IC3C.+IN, R21.2, R22.2
- net N$6: now also IC2A.-IN, IC2A.OUT, R6.1; no longer IC1D.-IN, R8.2, R9.1
- net N$7: now also IC2B.-IN, IC2B.OUT, R7.1; no longer IC3C.-IN, R23.2, R24.1
- net N$8: now also R5.2, R6.2; no longer R11.2, R12.2
- net N$9: now also R7.2, R8.1; no longer R13.2, R14.1
- net REF: now also X1-1.S
Other:
- note added: "A"
- note removed: "D"
- moved on the sheet: C1, C2, C3, IC1A, IC1B, IC1C, IC2A, IC2B, IC2C, IC3A, IC3B, IC3C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

Commit message: Revert "Fixed wiring"
This reverts commit 887158206b74e515af25e9af216689274ec85624.
Parts:
- added R13: 10k, rcl:R-US_R0603
Connections:
- net CH0: now also R1.1
- net CH1: now also R5.1
- net CH2: now also R9.1
- net GND: now also R13.2; no longer R1.1, R5.1, R9.1
- net REF: now also R13.1
Changed lines of the file:
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@@
 <part name="+3V1" library="supply1" library_urn="urn:adsk.eagle:library:371" deviceset="+3V3" device=""/>
 <part name="X1" library="Rembrandt Electronics - JST XH Connectors v1-0" deviceset="JST-XH-04-PIN" device="-LONG-PAD"/>
-<part name="GND1" library="supply1" library_urn="urn:adsk.eagle:library:371" deviceset="GND" device=""/>
-<part name="GND2" library="supply1" library_urn="urn:adsk.eagle:library:371" deviceset="GND" device=""/>
-<part name="GND3" library="supply1" library_urn="urn:adsk.eagle:library:371" deviceset="GND" device=""/>
+<part name="R13" library="rcl" library_urn="urn:adsk.eagle:library:334" deviceset="R-US_" device="R0603" package3d_urn="urn:adsk.eagle:package:23555/3" value="10k"/>
 </parts>
 <sheets>
@@
 <attribute name="NAME" x="205.74" y="57.658" size="1.524" layer="95"/>
 </instance>
-<instance part="GND1" gate="1" x="60.96" y="162.56" smashed="yes">
-<attribute name="VALUE" x="58.42" y="160.02" size="1.778" layer="96"/>
-</instance>
-<instance part="GND2" gate="1" x="60.96" y="111.76" smashed="yes">
-<attribute name="VALUE" x="58.42" y="109.22" size="1.778" layer="96"/>
-</instance>
-<instance part="GND3" gate="1" x="60.96" y="60.96" smashed="yes">
-<attribute name="VALUE" x="58.42" y="58.42" size="1.778" layer="96"/>
+<instance part="R13" gate="G$1" x="162.56" y="149.86" smashed="yes">
+<attribute name="NAME" x="158.75" y="151.3586" size="1.778" layer="95"/>
+<attribute name="VALUE" x="158.75" y="146.558" size="1.778" layer="96"/>
 </instance>
 </instances>
@@
 <wire x1="170.18" y1="116.84" x2="170.18" y2="149.86" width="0.1524" layer="91"/>
 <wire x1="170.18" y1="149.86" x2="180.34" y2="149.86" width="0.1524" layer="91"/>
+<pinref part="R13" gate="G$1" pin="2"/>
+<wire x1="170.18" y1="149.86" x2="167.64" y2="149.86" width="0.1524" layer="91"/>
+<junction x="170.18" y="149.86"/>
 </segment>
 <segment>
@@
 <junction x="187.96" y="83.82"/>
 </segment>
-<segment>
-<pinref part="GND1" gate="1" pin="GND"/>
-<wire x1="60.96" y1="165.1" x2="60.96" y2="167.64" width="0.1524" layer="91"/>
-<pinref part="R1" gate="G$1" pin="1"/>
-<wire x1="60.96" y1="167.64" x2="63.5" y2="167.64" width="0.1524" layer="91"/>
-</segment>
-<segment>
-<pinref part="GND2" gate="1" pin="GND"/>
-<wire x1="60.96" y1="114.3" x2="60.96" y2="116.84" width="0.1524" layer="91"/>
-<pinref part="R5" gate="G$1" pin="1"/>
-<wire x1="60.96" y1="116.84" x2="63.5" y2="116.84" width="0.1524" layer="91"/>
-</segment>
-<segment>
-<pinref part="GND3" gate="1" pin="GND"/>
-<wire x1="60.96" y1="63.5" x2="60.96" y2="66.04" width="0.1524" layer="91"/>
-<pinref part="R9" gate="G$1" pin="1"/>
-<wire x1="60.96" y1="66.04" x2="63.5" y2="66.04" width="0.1524" layer="91"/>
-</segment>
 </net>
 <net name="+3V3" class="0">
@@
 <segment>
 <pinref part="IC1" gate="A" pin="+IN"/>
+<wire x1="22.86" y1="160.02" x2="25.4" y2="160.02" width="0.1524" layer="91"/>
 <label x="22.86" y="160.02" size="1.27" layer="95" rot="R180" xref="yes"/>
-<wire x1="22.86" y1="160.02" x2="27.94" y2="160.02" width="0.1524" layer="91"/>
+<pinref part="R1" gate="G$1" pin="1"/>
+<wire x1="25.4" y1="160.02" x2="27.94" y2="160.02" width="0.1524" layer="91"/>
+<wire x1="63.5" y1="167.64" x2="25.4" y2="167.64" width="0.1524" layer="91"/>
+<wire x1="25.4" y1="167.64" x2="25.4" y2="160.02" width="0.1524" layer="91"/>
+<junction x="25.4" y="160.02"/>
 </segment>
 <segment>
@@
 <label x="22.86" y="83.82" size="1.27" layer="95" rot="R180" xref="yes"/>
 <pinref part="IC2" gate="B" pin="+IN"/>
+</segment>
+<segment>
+<pinref part="R13" gate="G$1" pin="1"/>
+<wire x1="154.94" y1="149.86" x2="157.48" y2="149.86" width="0.1524" layer="91"/>
+<label x="154.94" y="149.86" size="1.016" layer="95" rot="R180" xref="yes"/>
 </segment>
 <segment>
@@
 <segment>
 <pinref part="IC2" gate="A" pin="+IN"/>
+<wire x1="22.86" y1="109.22" x2="25.4" y2="109.22" width="0.1524" layer="91"/>
 <label x="22.86" y="109.22" size="1.27" layer="95" rot="R180" xref="yes"/>
-<wire x1="22.86" y1="109.22" x2="27.94" y2="109.22" width="0.1524" layer="91"/>
+<pinref part="R5" gate="G$1" pin="1"/>
+<wire x1="25.4" y1="109.22" x2="27.94" y2="109.22" width="0.1524" layer="91"/>
+<wire x1="63.5" y1="116.84" x2="25.4" y2="116.84" width="0.1524" layer="91"/>
+<wire x1="25.4" y1="116.84" x2="25.4" y2="109.22" width="0.1524" layer="91"/>
+<junction x="25.4" y="109.22"/>
 </segment>
 <segment>
@@
 <segment>
 <pinref part="IC3" gate="A" pin="+IN"/>
+<wire x1="22.86" y1="58.42" x2="25.4" y2="58.42" width="0.1524" layer="91"/>
 <label x="22.86" y="58.42" size="1.27" layer="95" rot="R180" xref="yes"/>
-<wire x1="22.86" y1="58.42" x2="27.94" y2="58.42" width="0.1524" layer="91"/>
+<pinref part="R9" gate="G$1" pin="1"/>
+<wire x1="25.4" y1="58.42" x2="27.94" y2="58.42" width="0.1524" layer="91"/>
+<wire x1="63.5" y1="66.04" x2="25.4" y2="66.04" width="0.1524" layer="91"/>
+<wire x1="25.4" y1="66.04" x2="25.4" y2="58.42" width="0.1524" layer="91"/>
+<junction x="25.4" y="58.42"/>
 </segment>
 <segment>
@@
 packages will not be understood (or retained) with this version.
 </note>
+<note version="8.4" severity="warning">
+Since Version 8.4, EAGLE supports properties for SPICE simulation.
+Probes in schematics and SPICE mapping objects found in parts and library devices
+will not be understood with this version. Update EAGLE to the latest version
+for full support of SPICE simulation.
+</note>
 </compatibility>

Commit message: Fixed wiring
Made sure it's a differential amplifier!
Removed R13.
Parts:
- removed R13: 10k, rcl:R-US_R0603
Connections:
- net CH0: no longer R1.1
- net CH1: no longer R5.1
- net CH2: no longer R9.1
- net GND: now also R1.1, R5.1, R9.1; no longer R13.2
- net REF: no longer R13.1
Changed lines of the file:
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@@
 <part name="+3V1" library="supply1" library_urn="urn:adsk.eagle:library:371" deviceset="+3V3" device=""/>
 <part name="X1" library="Rembrandt Electronics - JST XH Connectors v1-0" deviceset="JST-XH-04-PIN" device="-LONG-PAD"/>
-<part name="R13" library="rcl" library_urn="urn:adsk.eagle:library:334" deviceset="R-US_" device="R0603" package3d_urn="urn:adsk.eagle:package:23555/3" value="10k"/>
+<part name="GND1" library="supply1" library_urn="urn:adsk.eagle:library:371" deviceset="GND" device=""/>
+<part name="GND2" library="supply1" library_urn="urn:adsk.eagle:library:371" deviceset="GND" device=""/>
+<part name="GND3" library="supply1" library_urn="urn:adsk.eagle:library:371" deviceset="GND" device=""/>
 </parts>
 <sheets>
@@
 <attribute name="NAME" x="205.74" y="57.658" size="1.524" layer="95"/>
 </instance>
-<instance part="R13" gate="G$1" x="162.56" y="149.86" smashed="yes">
-<attribute name="NAME" x="158.75" y="151.3586" size="1.778" layer="95"/>
-<attribute name="VALUE" x="158.75" y="146.558" size="1.778" layer="96"/>
+<instance part="GND1" gate="1" x="60.96" y="162.56" smashed="yes">
+<attribute name="VALUE" x="58.42" y="160.02" size="1.778" layer="96"/>
+</instance>
+<instance part="GND2" gate="1" x="60.96" y="111.76" smashed="yes">
+<attribute name="VALUE" x="58.42" y="109.22" size="1.778" layer="96"/>
+</instance>
+<instance part="GND3" gate="1" x="60.96" y="60.96" smashed="yes">
+<attribute name="VALUE" x="58.42" y="58.42" size="1.778" layer="96"/>
 </instance>
 </instances>
@@
 <wire x1="170.18" y1="116.84" x2="170.18" y2="149.86" width="0.1524" layer="91"/>
 <wire x1="170.18" y1="149.86" x2="180.34" y2="149.86" width="0.1524" layer="91"/>
-<pinref part="R13" gate="G$1" pin="2"/>
-<wire x1="170.18" y1="149.86" x2="167.64" y2="149.86" width="0.1524" layer="91"/>
-<junction x="170.18" y="149.86"/>
 </segment>
 <segment>
@@
 <junction x="187.96" y="83.82"/>
 </segment>
+<segment>
+<pinref part="GND1" gate="1" pin="GND"/>
+<wire x1="60.96" y1="165.1" x2="60.96" y2="167.64" width="0.1524" layer="91"/>
+<pinref part="R1" gate="G$1" pin="1"/>
+<wire x1="60.96" y1="167.64" x2="63.5" y2="167.64" width="0.1524" layer="91"/>
+</segment>
+<segment>
+<pinref part="GND2" gate="1" pin="GND"/>
+<wire x1="60.96" y1="114.3" x2="60.96" y2="116.84" width="0.1524" layer="91"/>
+<pinref part="R5" gate="G$1" pin="1"/>
+<wire x1="60.96" y1="116.84" x2="63.5" y2="116.84" width="0.1524" layer="91"/>
+</segment>
+<segment>
+<pinref part="GND3" gate="1" pin="GND"/>
+<wire x1="60.96" y1="63.5" x2="60.96" y2="66.04" width="0.1524" layer="91"/>
+<pinref part="R9" gate="G$1" pin="1"/>
+<wire x1="60.96" y1="66.04" x2="63.5" y2="66.04" width="0.1524" layer="91"/>
+</segment>
 </net>
 <net name="+3V3" class="0">
@@
 <segment>
 <pinref part="IC1" gate="A" pin="+IN"/>
-<wire x1="22.86" y1="160.02" x2="25.4" y2="160.02" width="0.1524" layer="91"/>
 <label x="22.86" y="160.02" size="1.27" layer="95" rot="R180" xref="yes"/>
-<pinref part="R1" gate="G$1" pin="1"/>
-<wire x1="25.4" y1="160.02" x2="27.94" y2="160.02" width="0.1524" layer="91"/>
-<wire x1="63.5" y1="167.64" x2="25.4" y2="167.64" width="0.1524" layer="91"/>
-<wire x1="25.4" y1="167.64" x2="25.4" y2="160.02" width="0.1524" layer="91"/>
-<junction x="25.4" y="160.02"/>
+<wire x1="22.86" y1="160.02" x2="27.94" y2="160.02" width="0.1524" layer="91"/>
 </segment>
 <segment>
@@
 <label x="22.86" y="83.82" size="1.27" layer="95" rot="R180" xref="yes"/>
 <pinref part="IC2" gate="B" pin="+IN"/>
-</segment>
-<segment>
-<pinref part="R13" gate="G$1" pin="1"/>
-<wire x1="154.94" y1="149.86" x2="157.48" y2="149.86" width="0.1524" layer="91"/>
-<label x="154.94" y="149.86" size="1.016" layer="95" rot="R180" xref="yes"/>
 </segment>
 <segment>
@@
 <segment>
 <pinref part="IC2" gate="A" pin="+IN"/>
-<wire x1="22.86" y1="109.22" x2="25.4" y2="109.22" width="0.1524" layer="91"/>
 <label x="22.86" y="109.22" size="1.27" layer="95" rot="R180" xref="yes"/>
-<pinref part="R5" gate="G$1" pin="1"/>
-<wire x1="25.4" y1="109.22" x2="27.94" y2="109.22" width="0.1524" layer="91"/>
-<wire x1="63.5" y1="116.84" x2="25.4" y2="116.84" width="0.1524" layer="91"/>
-<wire x1="25.4" y1="116.84" x2="25.4" y2="109.22" width="0.1524" layer="91"/>
-<junction x="25.4" y="109.22"/>
+<wire x1="22.86" y1="109.22" x2="27.94" y2="109.22" width="0.1524" layer="91"/>
 </segment>
 <segment>
@@
 <segment>
 <pinref part="IC3" gate="A" pin="+IN"/>
-<wire x1="22.86" y1="58.42" x2="25.4" y2="58.42" width="0.1524" layer="91"/>
 <label x="22.86" y="58.42" size="1.27" layer="95" rot="R180" xref="yes"/>
-<pinref part="R9" gate="G$1" pin="1"/>
-<wire x1="25.4" y1="58.42" x2="27.94" y2="58.42" width="0.1524" layer="91"/>
-<wire x1="63.5" y1="66.04" x2="25.4" y2="66.04" width="0.1524" layer="91"/>
-<wire x1="25.4" y1="66.04" x2="25.4" y2="58.42" width="0.1524" layer="91"/>
-<junction x="25.4" y="58.42"/>
+<wire x1="22.86" y1="58.42" x2="27.94" y2="58.42" width="0.1524" layer="91"/>
 </segment>
 <segment>
@@
 packages will not be understood (or retained) with this version.
 </note>
-<note version="8.4" severity="warning">
-Since Version 8.4, EAGLE supports properties for SPICE simulation.
-Probes in schematics and SPICE mapping objects found in parts and library devices
-will not be understood with this version. Update EAGLE to the latest version
-for full support of SPICE simulation.
-</note>
 </compatibility>
